Commit message: implemented on triggers

File: resources/urdf/pr2_kinematic_tree.urdf (robot description, URDF)
Before this commit: robot pr2, 102 links, 101 joints
Links:
- removed link l_gripper_l_finger_tip_frame
- removed link odom_combined
- removed link odom_x_frame
- removed link odom_y_frame
- removed link r_gripper_l_finger_tip_frame
- link base_footprint: mass 1 -> None; geometry 
- link base_link: geometry collision box size=0.05 0.05 0.05; visual box size=0.05 0.05 0.05
- link bl_caster_l_wheel_link: geometry collision cylinder length=0.034 radius=0.074792; visual box size=0.05 0.05 0.05
- link bl_caster_r_wheel_link: geometry collision cylinder length=0.034 radius=0.074792; visual box size=0.05 0.05 0.05
- link bl_caster_rotation_link: geometry collision box size=0.05 0.05 0.05; visual box size=0.05 0.05 0.05
- link br_caster_l_wheel_link: geometry collision cylinder length=0.034 radius=0.074792; visual box size=0.05 0.05 0.05
- link br_caster_r_wheel_link: geometry collision cylinder length=0.034 radius=0.074792; visual box size=0.05 0.05 0.05
- link br_caster_rotation_link: geometry collision box size=0.05 0.05 0.05; visual box size=0.05 0.05 0.05
- link fl_caster_l_wheel_link: geometry collision cylinder length=0.034 radius=0.074792; visual box size=0.05 0.05 0.05
- link fl_caster_r_wheel_link: geometry collision cylinder length=0.034 radius=0.074792; visual box size=0.05 0.05 0.05
- link fl_caster_rotation_link: geometry collision box size=0.05 0.05 0.05; visual box size=0.05 0.05 0.05
- link fr_caster_l_wheel_link: geometry collision cylinder length=0.034 radius=0.074792; visual box size=0.05 0.05 0.05
- link fr_caster_r_wheel_link: geometry collision cylinder length=0.034 radius=0.074792; visual box size=0.05 0.05 0.05
- link fr_caster_rotation_link: geometry collision box size=0.05 0.05 0.05; visual box size=0.05 0.05 0.05
- link head_mount_kinect_ir_link: mass 0.1 -> None; geometry 
- link head_mount_kinect_rgb_link: mass 0.1 -> None; geometry 
- link head_mount_link: mass 0.1 -> None; geometry 
- link head_mount_prosilica_link: mass 0.1 -> None; geometry 
- link head_pan_link: geometry collision box size=0.05 0.05 0.05; visual box size=0.05 0.05 0.05
- link head_plate_frame: mass 0.01 -> None; geometry 
- link head_tilt_link: geometry collision box size=0.05 0.05 0.05; visual box size=0.05 0.05 0.05
- link l_elbow_flex_link: geometry collision box size=0.05 0.05 0.05; visual box size=0.05 0.05 0.05
- link l_force_torque_link: geometry collision cylinder length=0.0356 radius=0.0225; visual cylinder length=0.0356 radius=0.0225
- link l_forearm_link: geometry collision box size=0.05 0.05 0.05; visual box size=0.05 0.05 0.05
- link l_forearm_roll_link: geometry collision box size=0.05 0.05 0.05; visual box size=0.05 0.05 0.05
- link l_gripper_l_finger_link: geometry collision box size=0.05 0.05 0.05; visual box size=0.05 0.05 0.05
- link l_gripper_l_finger_tip_link: geometry collision box size=0.05 0.05 0.05; visual box size=0.05 0.05 0.05
- link l_gripper_motor_accelerometer_link: mass 0.001 -> None; geometry 
- link l_gripper_palm_link: geometry collision box size=0.05 0.05 0.05; visual box size=0.05 0.05 0.05
- link l_gripper_r_finger_link: geometry collision box size=0.05 0.05 0.05; visual box size=0.05 0.05 0.05
- link l_gripper_r_finger_tip_link: geometry collision box size=0.05 0.05 0.05; visual box size=0.05 0.05 0.05
- link l_shoulder_lift_link: geometry collision box size=0.05 0.05 0.05; visual box size=0.05 0.05 0.05
- link l_shoulder_pan_link: geometry collision box size=0.05 0.05 0.05; visual box size=0.05 0.05 0.05
- link l_upper_arm_link: geometry collision box size=0.05 0.05 0.05; visual box size=0.05 0.05 0.05
- link l_upper_arm_roll_link: geometry collision box size=0.05 0.05 0.05; visual box size=0.05 0.05 0.05
- link l_wrist_flex_link: geometry collision box size=0.05 0.05 0.05; visual box size=0.05 0.05 0.05
- link l_wrist_roll_link: geometry collision box size=0.05 0.05 0.05; visual box size=0.05 0.05 0.05
- link laser_tilt_mount_link: geometry collision box size=0.05 0.05 0.05; visual box size=0.05 0.05 0.05
- link r_elbow_flex_link: geometry collision box size=0.05 0.05 0.05; visual box size=0.05 0.05 0.05
- link r_forearm_link: geometry collision box size=0.05 0.05 0.05; visual box size=0.05 0.05 0.05
- link r_forearm_roll_link: geometry collision box size=0.05 0.05 0.05; visual box size=0.05 0.05 0.05
- link r_gripper_l_finger_link: geometry collision box size=0.05 0.05 0.05; visual box size=0.05 0.05 0.05
- link r_gripper_l_finger_tip_link: geometry collision box size=0.05 0.05 0.05; visual box size=0.05 0.05 0.05
- link r_gripper_motor_accelerometer_link: mass 0.001 -> None; geometry 
- link r_gripper_palm_link: geometry collision box size=0.05 0.05 0.05; visual box size=0.05 0.05 0.05
- link r_gripper_r_finger_link: geometry collision box size=0.05 0.05 0.05; visual box size=0.05 0.05 0.05
- link r_gripper_r_finger_tip_link: geometry collision box size=0.05 0.05 0.05; visual box size=0.05 0.05 0.05
- link r_shoulder_lift_link: geometry collision box size=0.05 0.05 0.05; visual box size=0.05 0.05 0.05
- link r_shoulder_pan_link: geometry collision box size=0.05 0.05 0.05; visual box size=0.05 0.05 0.05
- link r_upper_arm_link: geometry collision box size=0.05 0.05 0.05; visual box size=0.05 0.05 0.05
- link r_upper_arm_roll_link: geometry collision box size=0.05 0.05 0.05; visual box size=0.05 0.05 0.05
- link r_wrist_flex_link: geometry collision box size=0.05 0.05 0.05; visual box size=0.05 0.05 0.05
- link r_wrist_roll_link: geometry collision box size=0.05 0.05 0.05; visual box size=0.05 0.05 0.05
- link torso_lift_link: geometry collision box size=0.05 0.05 0.05; visual box size=0.05 0.05 0.05
Joints:
- removed joint l_gripper_joint
- removed joint odom_x_joint
- removed joint odom_y_joint
- removed joint odom_z_joint
- removed joint r_gripper_joint
- joint l_gripper_l_finger_tip_joint: mimic (none) -> joint=l_gripper_l_finger_joint multiplier=1 offset=0
- joint l_gripper_r_finger_joint: mimic (none) -> joint=l_gripper_l_finger_joint multiplier=1 offset=0
- joint l_gripper_r_finger_tip_joint: mimic (none) -> joint=l_gripper_l_finger_joint multiplier=1 offset=0
- joint r_gripper_l_finger_tip_joint: mimic (none) -> joint=r_gripper_l_finger_joint multiplier=1 offset=0
- joint r_gripper_r_finger_joint: mimic (none) -> joint=r_gripper_l_finger_joint multiplier=1 offset=0
- joint r_gripper_r_finger_tip_joint: mimic (none) -> joint=r_gripper_l_finger_joint multiplier=1 offset=0
- joint r_shoulder_lift_joint: limit lower=-0.5236 upper=1.3963 effort=30 velocity=2.082 -> lower=-0.5236 upper=1.3963 effort=30 velocity=0.2
- joint r_shoulder_pan_joint: limit lower=-2.2853981634 upper=0.714601836603 effort=30 velocity=2.088 -> lower=-2.2853981634 upper=0.714601836603 effort=30 velocity=0.15
