Commit message: Tiago test and reset fix

File: pycram/resources/robots/tiago_dual.urdf (robot description, URDF)
Before this commit: robot tiago_dual, 69 links, 68 joints
Links:
- link base_link: geometry collision mesh filename=package://pmb2_description/meshes/base/base_collision.dae; visual mesh filename=package://pmb2_description/meshes/base/base.stl
